File: aggregat02-iocontrols/aggregat02-iocontrols.sch (KiCad schematic (older format))
At the start: 69 parts, among them Q2 Q_NPN_BEC

Commit message: v1.0"
Parts:
- added J1, J2: Conn_01x04, Connector_PinHeader_2.54mm:PinHeader_1x04_P2.54mm_Vertical, symbol Connector_Generic:Conn_01x04
- added J10, J11, J12, J13, J14, J19, J4, J5, J6, J7, J8, J9: Conn_01x01, Connector_PinHeader_2.54mm:PinHeader_1x01_P2.54mm_Vertical, symbol Connector_Generic:Conn_01x01
- added J15, J16: Conn_01x15, Connector_Molex:Molex_PicoBlade_53047-1510_1x15_P1.25mm_Vertical, symbol Connector_Generic:Conn_01x15
- added J17: Conn_01x03, Connector_PinHeader_2.54mm:PinHeader_1x02_P2.54mm_Vertical, symbol Connector_Generic:Conn_01x02
- added J18: Conn_01x03, Connector_Molex:Molex_PicoBlade_53047-0310_1x03_P1.25mm_Vertical, symbol Connector_Generic:Conn_01x03
- added J3: Conn_01x08, Connector_PinHeader_2.54mm:PinHeader_1x08_P2.54mm_Vertical, symbol Connector_Generic:Conn_01x08
- added LD11, LD12, LD21, LD22, LD31, LD32, LD_MTR1: LED, LED_THT:LED_D3.0mm, symbol Device:LED
- added Q1, Q3, Q4, Q5, Q6, Q7, Q8: Q_NPN_BEC, Package_TO_SOT_SMD:SOT-23, symbol Device:Q_NPN_BEC
- added R42, R45, R48, R51, R54, R57, R60: R 47k 1% 1/8, Resistor_SMD:R_0805_2012Metric_Pad1.15x1.40mm_HandSolder, symbol Device:R
- added R43, R46, R49, R52, R55, R58, R61: R 100k 1% 1/8, Resistor_SMD:R_0805_2012Metric_Pad1.15x1.40mm_HandSolder, symbol Device:R
- added R44, R47, R50, R53, R56, R59, R62: R 270 1% 1/8, Resistor_SMD:R_0805_2012Metric_Pad1.15x1.40mm_HandSolder, symbol Device:R
- R39: value R -> R 270 1% 1/8
- R40: value R 270 1% 1/8 -> R 47k 1% 1/8
- renumbered D1 to LD_PWR1
Connections:
- net labels added: LED11, LED12, LED21, LED22, LED31, LED32, LED_MOTOR, LED_PWR
- net labels removed: LED_1
- wire segments 97 -> 134
Other:
- moved on the sheet: C1, C10, C11, C12, C13, C14, C15, C16, C17, C18, C19, C2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

Commit message: fixes
Connections:
- no-connect marks 0 -> 1
Changed lines of the file:
@@
 L power:GNDREF #PWR0142
 U 1 1 5F86F99F
-P 7150 5750
-F 0 "#PWR0142" H 7150 5500 50  0001 C CNN
-F 1 "GNDREF" H 7155 5577 50  0000 C CNN
-F 2 "" H 7150 5750 50  0001 C CNN
-F 3 "" H 7150 5750 50  0001 C CNN
-	1    7150 5750
+P 7200 5450
+F 0 "#PWR0142" H 7200 5200 50  0001 C CNN
+F 1 "GNDREF" H 7205 5277 50  0000 C CNN
+F 2 "" H 7200 5450 50  0001 C CNN
+F 3 "" H 7200 5450 50  0001 C CNN
+	1    7200 5450
 	1    0    0    -1
 $EndComp
-Wire Wire Line
-	6550 5750 7150 5750
 Wire Wire Line
 	4800 6050 5500 6050
@@
 Text GLabel 6550 5850 2    50   Input ~ 0
 LED11
-Text GLabel 6550 5350 2    50   Input ~ 0
+Text GLabel 6550 5550 2    50   Input ~ 0
 SW_CENTER
-Text GLabel 6550 5450 2    50   Input ~ 0
+Text GLabel 6550 5650 2    50   Input ~ 0
 SW_PLUS1
-Text GLabel 6550 5550 2    50   Input ~ 0
+Text GLabel 6550 5750 2    50   Input ~ 0
 SW_PLUS2
 $Comp
@@
 Text GLabel 8150 6000 0    50   Input ~ 0
 SW_NRST
+Wire Wire Line
+	6550 5450 7200 5450
+NoConn ~ 6550 5350
 $EndSCHEMATC

Commit message: v1.2
Parts:
- removed J18: Conn_01x03, Connector_Molex:Molex_PicoBlade_53047-0310_1x03_P1.25mm_Vertical, symbol Connector_Generic:Conn_01x03
- removed J8: Conn_01x01, Connector_PinHeader_2.54mm:PinHeader_1x01_P2.54mm_Vertical, symbol Connector_Generic:Conn_01x01
- CN1: renamed from J15; footprint Connector_Molex:Molex_PicoBlade_53047-1510_1x15_P1.25mm_Vertical -> Connector_PinHeader_2.54mm:PinHeader_1x15_P2.54mm_Vertical
- CN2: renamed from J16; footprint Connector_Molex:Molex_PicoBlade_53047-1510_1x15_P1.25mm_Vertical -> Connector_PinHeader_2.54mm:PinHeader_1x15_P2.54mm_Vertical
- renumbered J19 to NRST1
Connections:
- wire segments 134 -> 132
Changed lines of the file:
@@
 	8100 2000 8250 2000
-$Comp
-L Connector_Generic:Conn_01x01 J8
-U 1 1 5F5F18B7
-P 9250 1350
-F 0 "J8" H 9330 1392 50  0000 L CNN
-F 1 "Conn_01x01" H 9330 1301 50  0000 L CNN
-F 2 "Connector_PinHeader_2.54mm:PinHeader_1x01_P2.54mm_Vertical" H 9250 1350 50  0001 C CNN
-F 3 "~" H 9250 1350 50  0001 C CNN
-	1    9250 1350
-	-1   0    0    1
-$EndComp
 $Comp
 L Connector_Generic:Conn_01x01 J9
@@
 $EndComp
 Wire Wire Line
-	9450 1150 9450 1350
-Wire Wire Line
 	7300 2200 7300 2400
 $Comp
@@
 SW_CENTER
 $Comp
-L Connector_Generic:Conn_01x15 J15
-U 1 1 5F7AA3DE
-P 5700 5650
-F 0 "J15" H 5780 5692 50  0000 L CNN
-F 1 "Conn_01x15" H 5780 5601 50  0000 L CNN
-F 2 "Connector_Molex:Molex_PicoBlade_53047-1510_1x15_P1.25mm_Vertical" H 5700 5650 50  0001 C CNN
-F 3 "~" H 5700 5650 50  0001 C CNN
-	1    5700 5650
-	1    0    0    -1
-$EndComp
-$Comp
-L Connector_Generic:Conn_01x15 J16
-U 1 1 5F7ADAF9
-P 6350 5650
-F 0 "J16" H 6268 6567 50  0000 C CNN
-F 1 "Conn_01x15" H 6268 6476 50  0000 C CNN
-F 2 "Connector_Molex:Molex_PicoBlade_53047-1510_1x15_P1.25mm_Vertical" H 6350 5650 50  0001 C CNN
-F 3 "~" H 6350 5650 50  0001 C CNN
-	1    6350 5650
-	-1   0    0    -1
-$EndComp
-Text GLabel 5500 4950 0    50   Input ~ 0
-LED_MOTOR
-Text GLabel 5500 5050 0    50   Input ~ 0
-LED_PWR
-Text GLabel 5500 5150 0    50   Input ~ 0
-SW_CH_1
-Text GLabel 5500 5250 0    50   Input ~ 0
-SW_CH_2
-Text GLabel 5500 5350 0    50   Input ~ 0
-SW_CH_3
-Text GLabel 5500 5450 0    50   Input ~ 0
-SW_CH_4
-Text GLabel 5500 5550 0    50   Input ~ 0
-SW_ID_1
-Text GLabel 5500 5650 0    50   Input ~ 0
-SW_ID_2
-Text GLabel 5500 5750 0    50   Input ~ 0
-SW_ID_3
-Text GLabel 5500 5850 0    50   Input ~ 0
-SW_ID_4
+L Connector_Generic:Conn_01x02 J17
+U 1 1 5F8E90E9
+P 8350 5500
+F 0 "J17" H 8430 5492 50  0000 L CNN
+F 1 "Conn_01x03" H 8430 5401 50  0000 L CNN
+F 2 "Connector_PinHeader_2.54mm:PinHeader_1x02_P2.54mm_Vertical" H 8350 5500 50  0001 C CNN
+F 3 "~" H 8350 5500 50  0001 C CNN
+	1    8350 5500
+	1    0    0    -1
+$EndComp
+$Comp
+L power:GNDREF #PWR0145
+U 1 1 5F91115D
+P 8150 5600
+F 0 "#PWR0145" H 8150 5350 50  0001 C CNN
+F 1 "GNDREF" H 8155 5427 50  0000 C CNN
+F 2 "" H 8150 5600 50  0001 C CNN
+F 3 "" H 8150 5600 50  0001 C CNN
+	1    8150 5600
+	1    0    0    -1
+$EndComp
+$Comp
+L power:+3V3 #PWR0143
+U 1 1 5F8EDF90
+P 8150 5500
+F 0 "#PWR0143" H 8150 5350 50  0001 C CNN
+F 1 "+3V3" H 8165 5673 50  0000 C CNN
+F 2 "" H 8150 5500 50  0001 C CNN
+F 3 "" H 8150 5500 50  0001 C CNN
+	1    8150 5500
+	1    0    0    -1
+$EndComp
+$Comp
+L Connector_Generic:Conn_01x01 NRST1
+U 1 1 5F975D60
+P 8350 6000
+F 0 "NRST1" H 8430 6042 50  0000 L CNN
+F 1 "Conn_01x01" H 8430 5951 50  0000 L CNN
+F 2 "Connector_PinHeader_2.54mm:PinHeader_1x01_P2.54mm_Vertical" H 8350 6000 50  0001 C CNN
+F 3 "~" H 8350 6000 50  0001 C CNN
+	1    8350 6000
+	1    0    0    -1
+$EndComp
+Text GLabel 8150 6000 0    50   Input ~ 0
+SW_NRST
+Wire Wire Line
+	4800 6050 5500 6050
+Text GLabel 5500 6350 0    50   Input ~ 0
+SW_CFG_4
+Text GLabel 5500 6250 0    50   Input ~ 0
+SW_CFG_3
+Text GLabel 5500 6150 0    50   Input ~ 0
+SW_CFG_2
+Text GLabel 5500 5950 0    50   Input ~ 0
+SW_CFG_1
 $Comp
 L power:GNDREF #PWR0141
@@
 	1    0    0    -1
 $EndComp
-Text GLabel 5500 5950 0    50   Input ~ 0
-SW_CFG_1
-Text GLabel 5500 6150 0    50   Input ~ 0
-SW_CFG_2
-Text GLabel 5500 6250 0    50   Input ~ 0
-SW_CFG_3
-Text GLabel 5500 6350 0    50   Input ~ 0
-SW_CFG_4
+Text GLabel 5500 5850 0    50   Input ~ 0
+SW_ID_4
+Text GLabel 5500 5750 0    50   Input ~ 0
+SW_ID_3
+Text GLabel 5500 5650 0    50   Input ~ 0
+SW_ID_2
+Text GLabel 5500 5550 0    50   Input ~ 0
+SW_ID_1
+Text GLabel 5500 5450 0    50   Input ~ 0
+SW_CH_4
+Text GLabel 5500 5350 0    50   Input ~ 0
+SW_CH_3
+Text GLabel 5500 5250 0    50   Input ~ 0
+SW_CH_2
+Text GLabel 5500 5150 0    50   Input ~ 0
+SW_CH_1
+Text GLabel 5500 5050 0    50   Input ~ 0
+LED_PWR
+Text GLabel 5500 4950 0    50   Input ~ 0
+LED_MOTOR
+NoConn ~ 6550 5350
+Wire Wire Line
+	6550 5450 7200 5450
+Text GLabel 6550 5750 2    50   Input ~ 0
+SW_PLUS2
+Text GLabel 6550 5650 2    50   Input ~ 0
+SW_PLUS1
+Text GLabel 6550 5550 2    50   Input ~ 0
+SW_CENTER
+Text GLabel 6550 5850 2    50   Input ~ 0
+LED11
+Text GLabel 6550 5950 2    50   Input ~ 0
+LED12
+Text GLabel 6550 6050 2    50   Input ~ 0
+LED21
+Text GLabel 6550 6150 2    50   Input ~ 0
+LED22
+Text GLabel 6550 6250 2    50   Input ~ 0
+LED31
+Text GLabel 6550 6350 2    50   Input ~ 0
+LED32
+Text GLabel 6550 5250 2    50   Input ~ 0
+SW_CFG_8
+Text GLabel 6550 5150 2    50   Input ~ 0
+SW_CFG_7
+Text GLabel 6550 5050 2    50   Input ~ 0
+SW_CFG_6
+Text GLabel 6550 4950 2    50   Input ~ 0
+SW_CFG_5
 $Comp
 L power:GNDREF #PWR0142
@@
 	1    0    0    -1
 $EndComp
-Wire Wire Line
-	4800 6050 5500 6050
-Text GLabel 6550 4950 2    50   Input ~ 0
-SW_CFG_5
-Text GLabel 6550 5050 2    50   Input ~ 0
-SW_CFG_6
-Text GLabel 6550 5150 2    50   Input ~ 0
-SW_CFG_7
-Text GLabel 6550 5250 2    50   Input ~ 0
-SW_CFG_8
-Text GLabel 6550 6350 2    50   Input ~ 0
-LED32
-Text GLabel 6550 6250 2    50   Input ~ 0
-LED31
-Text GLabel 6550 6150 2    50   Input ~ 0
-LED22
-Text GLabel 6550 6050 2    50   Input ~ 0
-LED21
-Text GLabel 6550 5950 2    50   Input ~ 0
-LED12
-Text GLabel 6550 5850 2    50   Input ~ 0
-LED11
-Text GLabel 6550 5550 2    50   Input ~ 0
-SW_CENTER
-Text GLabel 6550 5650 2    50   Input ~ 0
-SW_PLUS1
-Text GLabel 6550 5750 2    50   Input ~ 0
-SW_PLUS2
-$Comp
-L Connector_Generic:Conn_01x02 J17
-U 1 1 5F8E90E9
-P 8350 5500
-F 0 "J17" H 8430 5492 50  0000 L CNN
-F 1 "Conn_01x03" H 8430 5401 50  0000 L CNN
-F 2 "Connector_PinHeader_2.54mm:PinHeader_1x02_P2.54mm_Vertical" H 8350 5500 50  0001 C CNN
-F 3 "~" H 8350 5500 50  0001 C CNN
-	1    8350 5500
-	1    0    0    -1
-$EndComp
-$Comp
-L power:GNDREF #PWR0145
-U 1 1 5F91115D
-P 8150 5600
-F 0 "#PWR0145" H 8150 5350 50  0001 C CNN
-F 1 "GNDREF" H 8155 5427 50  0000 C CNN
-F 2 "" H 8150 5600 50  0001 C CNN
-F 3 "" H 8150 5600 50  0001 C CNN
-	1    8150 5600
-	1    0    0    -1
-$EndComp
-$Comp
-L power:GNDREF #PWR0146
-U 1 1 5F9155C7
-P 9300 5600
-F 0 "#PWR0146" H 9300 5350 50  0001 C CNN
-F 1 "GNDREF" H 9305 5427 50  0000 C CNN
-F 2 "" H 9300 5600 50  0001 C CNN
-F 3 "" H 9300 5600 50  0001 C CNN
-	1    9300 5600
-	-1   0    0    1
-$EndComp
-$Comp
-L power:+3V3 #PWR0144
-U 1 1 5F8F6768
-P 9550 5500
-F 0 "#PWR0144" H 9550 5350 50  0001 C CNN
-F 1 "+3V3" H 9565 5673 50  0000 C CNN
-F 2 "" H 9550 5500 50  0001 C CNN
-F 3 "" H 9550 5500 50  0001 C CNN
-	1    9550 5500
-	1    0    0    -1
-$EndComp
-Text GLabel 9550 5700 0    50   Input ~ 0
-SW_NRST
-$Comp
-L power:+3V3 #PWR0143
-U 1 1 5F8EDF90
-P 8150 5500
-F 0 "#PWR0143" H 8150 5350 50  0001 C CNN
-F 1 "+3V3" H 8165 5673 50  0000 C CNN
-F 2 "" H 8150 5500 50  0001 C CNN
-F 3 "" H 8150 5500 50  0001 C CNN
-	1    8150 5500
-	1    0    0    -1
-$EndComp
-$Comp
-L Connector_Generic:Conn_01x03 J18
-U 1 1 5F8E9B09
-P 9750 5600
-F 0 "J18" H 9830 5642 50  0000 L CNN
-F 1 "Conn_01x03" H 9830 5551 50  0000 L CNN
-F 2 "Connector_Molex:Molex_PicoBlade_53047-0310_1x03_P1.25mm_Vertical" H 9750 5600 50  0001 C CNN
-F 3 "~" H 9750 5600 50  0001 C CNN
-	1    9750 5600
-	1    0    0    -1
-$EndComp
-Wire Wire Line
-	9550 5600 9300 5600
-$Comp
-L Connector_Generic:Conn_01x01 J19
-U 1 1 5F975D60
-P 8350 6000
-F 0 "J19" H 8430 6042 50  0000 L CNN
-F 1 "Conn_01x01" H 8430 5951 50  0000 L CNN
-F 2 "Connector_PinHeader_2.54mm:PinHeader_1x01_P2.54mm_Vertical" H 8350 6000 50  0001 C CNN
-F 3 "~" H 8350 6000 50  0001 C CNN
-	1    8350 6000
-	1    0    0    -1
-$EndComp
-Text GLabel 8150 6000 0    50   Input ~ 0
-SW_NRST
-Wire Wire Line
-	6550 5450 7200 5450
-NoConn ~ 6550 5350
+$Comp
+L Connector_Generic:Conn_01x15 CN1
+U 1 1 5F7AA3DE
+P 5700 5650
+F 0 "CN1" H 5780 5692 50  0000 L CNN
+F 1 "Conn_01x15" H 5780 5601 50  0000 L CNN
+F 2 "Connector_PinHeader_2.54mm:PinHeader_1x15_P2.54mm_Vertical" H 5700 5650 50  0001 C CNN
+F 3 "~" H 5700 5650 50  0001 C CNN
+	1    5700 5650
+	1    0    0    -1
+$EndComp
+$Comp
+L Connector_Generic:Conn_01x15 CN2
+U 1 1 5F7ADAF9
+P 6350 5650
+F 0 "CN2" H 6268 6567 50  0000 C CNN
+F 1 "Conn_01x15" H 6268 6476 50  0000 C CNN
+F 2 "Connector_PinHeader_2.54mm:PinHeader_1x15_P2.54mm_Vertical" H 6350 5650 50  0001 C CNN
+F 3 "~" H 6350 5650 50  0001 C CNN
+	1    6350 5650
+	-1   0    0    -1
+$EndComp
 $EndSCHEMATC
